File: Circuit/Main Board.kicad_pcb (KiCad board)
At the start: 2 copper layers, 120 x 120 mm, 200 parts, among them J1 Conn_Coaxial, J2 Conn_Coaxial, J3 Conn_Coaxial, J4 Conn_Coaxial, J5 Conn_01x02_Pin, J6 Conn_01x03_Pin, J7 Conn_01x02_Pin, J8 Conn_01x02_Pin, J9 Conn_01x05_Pin, K1 AGQ200A12, K2 AGQ200A12, K3 AGQ200A12, K4 AGQ200A12, K5 AGQ200A12, K6 AGQ200A12, K7 AGQ200A12, Q1 2N7002, Q2 TIP41C, Q3 TIP42C, Q4 TIP41C, Q5 TIP42C, Q6 TIP41C, Q7 TIP42C, U1 STM32G491CCUx, U10 OPA2197xD, U11 INA828D, U12 DG201, U13 OPA2197xD, U14 DG201, U15 OPA2376xxD, U16 INA828D, U17 DG201, U18 OPA2376xxD, U2 DG201, U3 OPA2197xD, U4 OPA2197xD, U5 OPA2197xD, U6 OPA2197xD, U7 ULN2003, U8 DG201, U9 OPA2376xxD, Y1 ECS-2520MV-xxx-xx

Commit message: Output job, Revision Box and reorganise
Parts:
- moved D6 2.54 mm to (80.0, 46.0)
- moved R87 2.54 mm to (80.0, 48.0)
Routing:
- net +12V: track 414.1 -> 417.6 mm
- net +3.3V: track 115.0 -> 112.4 mm
Other:
- board text added: "${COMMENT1} ${TITLE}"
- board text added: "Rev. ${REVISION}."
Changed lines of the file:
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@@
 	)
 	(paper "A4")
+	(title_block
+		(title "A1 Main Board")
+		(date "2026-05-02")
+		(rev "1")
+		(company "Harry Hill and Yuki Hoshino")
+		(comment 1 "LCR Meter")
+	)
 	(layers
 		(0 "F.Cu" signal)
@@
 	(footprint "LED_SMD:LED_0805_2012Metric"
 		(layer "F.Cu")
-		(at 77.47 45.974 180)
+		(at 80.01 45.974 180)
 		(descr "LED SMD 0805 (2012 Metric), square (rectangular) end terminal, IPC-7351 nominal, (Body size source: https://docs.google.com/spreadsheets/d/1BsfQQcO9C6DZCsRaXUlFlo91Tg2WpOkGARC1WS5S8t0/edit?usp=sharing), generated with kicad-footprint-generator")
 		(tags "LED")
@@
 	(footprint "Resistor_SMD:R_0805_2012Metric"
 		(layer "F.Cu")
-		(at 77.47 48.006 180)
+		(at 80.01 48.006 180)
 		(descr "Resistor SMD 0805 (2012 Metric), square (rectangular) end terminal, IPC-7351 nominal, (Body size source: IPC-SM-782 page 72, https://www.pcb-3d.com/wordpress/wp-content/uploads/ipc-sm-782a_amendment_1_and_2.pdf), generated with kicad-footprint-generator")
 		(tags "resistor")
@@
 		(tags "resistor")
 		(property "Reference" "R16"
-			(at 2.315 -0.061 180)
+			(at 0 -1.016 180)
 			(layer "F.SilkS")
 			(effects
@@
 		(tags "SOIC SO 16-pin-NSOP R-16 R-16-S D0016A M2B SO16 SOT109-1 751B SOIC_N narrow")
 		(property "Reference" "U7"
-			(at 0 5.588 0)
+			(at 0 -5.588 0)
 			(layer "F.SilkS")
 			(effects
@@
 					(thickness 0.15)
 				)
-				(justify right bottom)
+				(justify right top)
 			)
 		)
@@
 		)
 		(property "Value" "MountingHole"
-			(at -2.54 1.403187 0)
+			(at -0.078 0.105 0)
 			(layer "F.Fab")
 			(effects
@@
 	)
 	(gr_rect
+		(start 63.373 49.911)
+		(end 67.818 53.848)
+		(stroke
+			(width 0.1)
+			(type default)
+		)
+		(fill yes)
+		(layer "F.SilkS")
+	)
+	(gr_rect
+		(start 54.61 50.038)
+		(end 67.691 53.721)
+		(stroke
+			(width 0.5)
+			(type default)
+		)
+		(fill no)
+		(layer "F.SilkS")
+	)
+	(gr_rect
 		(start 41.6 42.56)
 		(end 161.6 162.56)
@@
 		(layer "User.1")
 	)
+	(gr_text "${COMMENT1}\n${TITLE}"
+		(at 55.118 44.958 0)
+		(layer "F.Mask")
+		(effects
+			(font
+				(size 1.5 1.5)
+				(thickness 0.2)
+				(bold yes)
+			)
+			(justify left top)
+		)
+	)
 	(gr_text "18"
 		(at 106.68 50.419 0)
@@
 		)
 	)
+	(gr_text "Rev. ${REVISION}."
+		(at 55.118 51.8795 0)
+		(layer "F.SilkS")
+		(effects
+			(font
+				(size 1.5 1.5)
+				(thickness 0.2)
+				(bold yes)
+			)
+			(justify left)
+		)
+	)
 	(gr_text "Serial"
 		(at 132.715 54.991 0)
@@
 	)
 	(gr_text "PWR"
-		(at 77.47 44.831 0)
+		(at 80.01 44.310499 0)
 		(layer "F.SilkS")
 		(effects
@@
 	)
 	(segment
+		(start 53.975 44.577)
+		(end 55.241 43.311)
+		(width 0.5)
+		(layer "F.Cu")
+		(net 10)
+	)
+	(segment
 		(start 153.035 136.525)
 		(end 153.355 136.205)
@@
 	)
 	(segment
-		(start 57.215 56.515)
-		(end 57.215 45.02)
-		(width 0.5)
-		(layer "F.Cu")
-		(net 10)
-	)
-	(segment
 		(start 104.14 47.4345)
 		(end 104.14 46.99)
@@
 	)
 	(segment
+		(start 55.241 43.311)
+		(end 102.366 43.311)
+		(width 0.5)
+		(layer "F.Cu")
+		(net 10)
+	)
+	(segment
 		(start 56.2991 102.860005)
 		(end 54.619995 102.860005)
@@
 	)
 	(segment
-		(start 104.14 45.085)
-		(end 104.14 46.99)
-		(width 0.5)
-		(layer "F.Cu")
-		(net 10)
-	)
-	(segment
 		(start 54.61 115.57)
 		(end 54.619995 115.560005)
@@
 	)
 	(segment
-		(start 58.924 43.311)
-		(end 102.366 43.311)
+		(start 45.72 56.515)
+		(end 57.215 56.515)
 		(width 0.5)
 		(layer "F.Cu")
@@
 	)
 	(segment
-		(start 45.72 56.515)
-		(end 57.215 56.515)
+		(start 104.14 45.085)
+		(end 104.14 46.99)
 		(width 0.5)
 		(layer "F.Cu")
@@
 	)
 	(segment
+		(start 53.975 56.515)
+		(end 53.975 44.577)
+		(width 0.5)
+		(layer "F.Cu")
+		(net 10)
+	)
+	(segment
 		(start 61.585005 140.960005)
 		(end 61.595 140.97)
@@
 	)
 	(segment
+		(start 102.366 43.311)
+		(end 104.14 45.085)
+		(width 0.5)
+		(layer "F.Cu")
+		(net 10)
+	)
+	(segment
 		(start 54.619995 121.92)
 		(end 54.619995 127.752005)
@@
 	)
 	(segment
-		(start 102.366 43.311)
-		(end 104.14 45.085)
-		(width 0.5)
-		(layer "F.Cu")
-		(net 10)
-	)
-	(segment
 		(start 70.055905 107.95)
 		(end 70.0659 107.959995)
@@
 		(net 10)
 	)
-	(segment
-		(start 57.215 45.02)
-		(end 58.924 43.311)
-		(width 0.5)
-		(layer "F.Cu")
-		(net 10)
-	)
 	(via
 		(at 54.61 102.87)
@@
 	)
 	(segment
-		(start 78.3825 48.006)
-		(end 78.3825 50.1885)
-		(width 0.2)
-		(layer "F.Cu")
-		(net 12)
-	)
-	(segment
 		(start 110.49 58.42)
 		(end 110.49 60.833)
@@
 	)
 	(segment
-		(start 114.554 81.026)
-		(end 114.554 78.565087)
+		(start 81.534 50.8)
+		(end 92.456 50.8)
 		(width 0.2)
 		(layer "F.Cu")
@@
 	)
 	(segment
-		(start 114.5075 61.976)
-		(end 114.5075 62.1835)
+		(start 114.554 81.026)
+		(end 114.554 78.565087)
 		(width 0.2)
 		(layer "F.Cu")
@@
 	)
 	(segment
-		(start 78.994 50.8)
-		(end 92.456 50.8)
+		(start 114.5075 61.976)
+		(end 114.5075 62.1835)
 		(width 0.2)
 		(layer "F.Cu")
@@
 	)
 	(segment
-		(start 92.456 50.8)
-		(end 92.915001 50.340999)
-		(width 0.2)
-		(layer "F.Cu")
-		(net 12)
-	)
-	(segment
 		(start 120.56 82.386)
 		(end 120.65 82.296)
@@
 	)
 	(segment
-		(start 78.3825 50.1885)
-		(end 78.994 50.8)
-		(width 0.2)
-		(layer "F.Cu")
-		(net 12)
-	)
-	(segment
 		(start 110.49 57.15)
 		(end 113.03 57.15)
@@
 	)
 	(segment
+		(start 92.456 50.8)
+		(end 92.915001 50.340999)
+		(width 0.2)
+		(layer "F.Cu")
+		(net 12)
+	)
+	(segment
 		(start 114.620001 81.346001)
 		(end 114.620001 81.092001)
@@
 	)
 	(segment
-		(start 92.915001 50.340999)
-		(end 92.915001 48.768)
-		(width 0.2)
-		(layer "F.Cu")
-		(net 12)
-	)
-	(segment
 		(start 114.62 83.312)
 		(end 114.62 81.28)
@@
 	)
 	(segment
+		(start 80.9225 50.1885)
+		(end 81.534 50.8)
+		(width 0.2)
+		(layer "F.Cu")
+		(net 12)
+	)
+	(segment
 		(start 101.6 55.88)
 		(end 109.22 55.88)
@@
 	)
 	(segment
+		(start 92.915001 50.340999)
+		(end 92.915001 48.768)
+		(width 0.2)
+		(layer "F.Cu")
+		(net 12)
+	)
+	(segment
 		(start 111.633 61.976)
 		(end 114.5075 61.976)
@@
 	)
 	(segment
+		(start 80.9225 48.006)
+		(end 80.9225 50.1885)
+		(width 0.2)
+		(layer "F.Cu")
+		(net 12)
+	)
+	(segment
 		(start 114.554 78.565087)
 		(end 115.083864 78.035223)
@@
 	)
 	(segment
-		(start 76.5575 48.006)
-		(end 76.5575 45.999001)
+		(start 79.0975 48.006)
+		(end 79.0975 45.999001)
 		(width 0.5)
 		(layer "F.Cu")
@@
 	)
 	(segment
-		(start 76.5575 45.999001)
-		(end 76.532499 45.974)
+		(start 79.0975 45.4785)
+		(end 79.072499 45.453499)
 		(width 0.5)
 		(layer "F.Cu")
