File: Circuit/Main Board.kicad_pcb (KiCad board)
At the start: 2 copper layers, 120 x 120 mm, 217 parts, among them J1 Conn_01x02_Pin, J2 Conn_Coaxial, J3 Conn_Coaxial, J4 Conn_Coaxial, J5 Conn_Coaxial, J6 Conn_01x03_Pin, J7 Conn_01x02_Pin, J8 Conn_01x02_Pin, J9 Conn_01x05_Pin, K1 AGQ200A12, K2 AGQ200A12, K3 AGQ200A12, K4 AGQ200A12, K5 AGQ200A12, K6 AGQ200A12, K7 AGQ200A12, Q1 2N7002, Q2 TIP41C, Q3 TIP42C, Q4 TIP41C, Q5 TIP42C, Q6 TIP41C, Q7 TIP42C, U1 STM32G491CCUx, U10 OPA2376xxD, U11 INA828D, U12 DG201, U13 OPA2197xD, U14 DG201, U15 OPA2376xxD, U16 INA828D, U17 DG201, U18 OPA2376xxD, U2 DG201, U3 OPA2197xD, U4 OPA2197xD, U5 OPA2197xD, U6 OPA2197xD, U7 ULN2003, U8 OPA2197xD, U9 DG201, Y1 ECS-2520MV-xxx-xx

Commit message: Adjustments
Parts:
- removed JP1: SolderJumper_2_Open, Jumper:SolderJumper-2_P1.3mm_Open_RoundedPad1.0x1.5mm
- added D15: BAV99, Package_TO_SOT_SMD:SOT-23, F.Cu at (141.0, 119.4)
- moved D5 2.84 mm to (146.1, 119.4), turned to 180 degrees
- turned K1 to -90 degrees
Connections:
- K1 pad 4: Net-(JP1-B) -> Net-(K1-Pad4)
- R29 pad 2: Net-(K1-Pad2) -> Net-(K1-Pad4)
- R30 pad 2: Net-(K1-Pad2) -> Net-(K1-Pad4)
- R31 pad 2: Net-(JP1-B) -> Net-(K1-Pad2)
- R32 pad 2: Net-(JP1-B) -> Net-(K1-Pad2)
- R40 pad 1: GUARD -> Net-(U8A--)
- U8 pad 2: GUARD -> Net-(U8A--)
Routing:
- net Net-(JP1-B): track 36.3 -> 0.00 mm
- net Net-(K1-Pad4): track 0.00 -> 19.9 mm
- net Net-(Q2-E): track 53.7 -> 66.2 mm
- net GUARD: track 550.9 -> 562.3 mm
- net /Signal Source/RELAY_DRIVE: track 11.9 -> 20.0 mm
- net /Auto-Balancing Bridge/TIA_SUM: track 176.0 -> 181.0 mm
- net Net-(K1-Pad2): track 20.2 -> 25.3 mm
- net Net-(D5-A): track 16.0 -> 20.9 mm
- net -18V: track 423.6 -> 427.2 mm
- net /Signal Source/Out: track 36.4 -> 32.9 mm
- net +18V: track 413.9 -> 416.6 mm
- net Net-(D5-K-Pad3): track 11.9 -> 9.41 mm
- net Net-(Q2-B): track 11.9 -> 9.47 mm
- net +12V: track 405.0 -> 403.0 mm
- net /Auto-Balancing Bridge/SEL_1k: track 86.0 -> 86.6 mm
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
Commit message: Final Touches
Parts:
- moved J9 10.2 mm to (96.5, 47.0), turned to 0 degrees
Connections:
- J9 pad 1: +18V -> -18V
- J9 pad 2: +12V -> GND
- J9 pad 4: GND -> +12V
- J9 pad 5: -18V -> +18V
Routing:
- net /Auto-Balancing Bridge/OUT+: track 174.8 -> 177.7 mm, vias 11 -> 12
