File: Circuit/Main Board.kicad_sch (KiCad schematic)
At the start: 9 parts, among them J1 Conn_Coaxial, J2 Conn_Coaxial, J3 Conn_Coaxial, J4 Conn_Coaxial, J5 Conn_01x02_Pin

Commit message: Output job, Revision Box and reorganise
Other:
- company: Harry and Yuki - EEE3 Instrumentation -> Harry Hill and Yuki Hoshino
- title: Interconnect -> Root
Changed lines of the file:
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@@
 	(paper "A4")
 	(title_block
-		(title "Interconnect")
-		(date "2026-03-02")
+		(title "Root")
+		(date "2026-05-02")
 		(rev "1.0")
-		(company "Harry and Yuki - EEE3 Instrumentation")
+		(company "Harry Hill and Yuki Hoshino")
+		(comment 1 "LCR Meter")
 	)
 	(text "LPOT\n"

Commit message: Input Protection Second Attempt
Parts:
- added D1, D2, D3: BAV199, Package_TO_SOT_SMD:SOT-23, symbol Diode:BAV99
- added R1, R2: 1k, Resistor_SMD:R_0805_2012Metric, symbol Device:R
- added R3, R4: 100k, Resistor_SMD:R_0805_2012Metric, symbol Device:R
- added R5: 50, Resistor_SMD:R_0805_2012Metric, symbol Device:R
- renumbered J5 to J1, J1 to J2, J2 to J3, J3 to J4, J4 to J5
Connections:
- net Auto-Balancing Bridge/In: now also D3.3 (K), R4.1
- net GND: now also D2.1 (K), D2.2 (A), D3.1 (K), D3.2 (A); no longer J2.2 (Ext), J3.2 (Ext)
- net Signal Source/Aux_Out: now also R5.1; no longer J1.1 (Pin_1)
- net Signal Source/Out: now also R3.1
- net Voltage Amplifier/In+: now also D1.3 (K), R1.1; no longer J3.1 (In)
- net Voltage Amplifier/In-: now also D2.3 (K), R2.2; no longer J4.1 (In)
- net GUARD renamed GUARD EXT
- net GUARD EXT: now also J2.2 (Ext), J3.2 (Ext)
- new net: J4.1 (In), R2.1, R4.2
- new net: J3.1 (In), R1.2, R3.2
- new net: J1.1 (Pin_1), R5.2
- new net +18V: D1.1 (K)
- new net -18V: D1.2 (A)
Other:
- moved on the sheet: J1, J2, J3, J4, J5

Commit message: New Resistor Selection Circuit
Changed lines of the file:
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@@
 		)
 		(pin "R_SEL_10k" input
-			(at 101.6 148.59 180)
+			(at 101.6 151.13 180)
 			(effects
 				(font
@@
 		)
 		(pin "R_SEL_1k" input
-			(at 101.6 151.13 180)
+			(at 101.6 148.59 180)
 			(effects
 				(font
