File: Circuit/currentamp.kicad_sch (KiCad schematic)
At the start: 21 parts, among them U16 INA828D, U17 DG201, U18 OPA2376xxD

Commit message: Output job, Revision Box and reorganise
Other:
- company: Harry and Yuki - EEE3 Instrumentation -> Harry Hill and Yuki Hoshino

Commit message: Input Protection Second Attempt
Parts:
- renumbered R76 to R80, R77 to R81, R78 to R82, R79 to R83, R80 to R84, R81 to R85, R82 to R86, R83 to R87, R84 to R88, R85 to R89, R86 to R90
Changed lines of the file:
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@@
 		(title "Current Amplifier")
 		(date "2026-05-02")
-		(rev "1.0")
+		(rev "0.1")
 		(company "Harry Hill and Yuki Hoshino")
 		(comment 1 "LCR Meter")
@@
 		(on_board yes)
 		(dnp no)
-		(property "Reference" "R81"
+		(property "Reference" "R85"
 			(at 139.7 73.66 90)
 			(effects
@@
 			(project "Main Board"
 				(path "/20aae4b7-3fb8-4924-82e8-1e7a29a313f8/2e1ccfa8-8bce-4bb4-9d3d-716156df4d18"
-					(reference "R81")
+					(reference "R85")
 					(unit 1)
 				)
@@
 		(dnp no)
 		(fields_autoplaced yes)
-		(property "Reference" "R85"
+		(property "Reference" "R89"
 			(at 237.49 57.1499 0)
 			(effects
@@
 			(project "Main Board"
 				(path "/20aae4b7-3fb8-4924-82e8-1e7a29a313f8/2e1ccfa8-8bce-4bb4-9d3d-716156df4d18"
-					(reference "R85")
+					(reference "R89")
 					(unit 1)
 				)
@@
 		(dnp no)
 		(fields_autoplaced yes)
-		(property "Reference" "#PWR0118"
+		(property "Reference" "#PWR0121"
 			(at 119.38 85.09 0)
 			(effects
@@
 			(project "Main Board"
 				(path "/20aae4b7-3fb8-4924-82e8-1e7a29a313f8/2e1ccfa8-8bce-4bb4-9d3d-716156df4d18"
-					(reference "#PWR0118")
+					(reference "#PWR0121")
 					(unit 1)
 				)
@@
 		(on_board yes)
 		(dnp no)
-		(property "Reference" "#PWR0117"
+		(property "Reference" "#PWR0120"
 			(at 38.1 54.61 0)
 			(effects
@@
 			(project "Main Board"
 				(path "/20aae4b7-3fb8-4924-82e8-1e7a29a313f8/2e1ccfa8-8bce-4bb4-9d3d-716156df4d18"
-					(reference "#PWR0117")
+					(reference "#PWR0120")
 					(unit 1)
 				)
@@
 		(dnp no)
 		(fields_autoplaced yes)
-		(property "Reference" "#PWR0126"
+		(property "Reference" "#PWR0129"
 			(at 265.43 124.46 0)
 			(effects
@@
 			(project "Main Board"
 				(path "/20aae4b7-3fb8-4924-82e8-1e7a29a313f8/2e1ccfa8-8bce-4bb4-9d3d-716156df4d18"
-					(reference "#PWR0126")
+					(reference "#PWR0129")
 					(unit 1)
 				)
@@
 		(on_board yes)
 		(dnp no)
-		(property "Reference" "R77"
+		(property "Reference" "R81"
 			(at 63.5 63.5 90)
 			(effects
@@
 			(project "Main Board"
 				(path "/20aae4b7-3fb8-4924-82e8-1e7a29a313f8/2e1ccfa8-8bce-4bb4-9d3d-716156df4d18"
-					(reference "R77")
+					(reference "R81")
 					(unit 1)
 				)
@@
 		(dnp no)
 		(fields_autoplaced yes)
-		(property "Reference" "R76"
+		(property "Reference" "R80"
 			(at 57.15 44.45 90)
 			(effects
@@
 			(project "Main Board"
 				(path "/20aae4b7-3fb8-4924-82e8-1e7a29a313f8/2e1ccfa8-8bce-4bb4-9d3d-716156df4d18"
-					(reference "R76")
+					(reference "R80")
 					(unit 1)
 				)
@@
 		(dnp no)
 		(fields_autoplaced yes)
-		(property "Reference" "#PWR0115"
+		(property "Reference" "#PWR0118"
 			(at 33.02 46.99 0)
 			(effects
@@
 			(project "Main Board"
 				(path "/20aae4b7-3fb8-4924-82e8-1e7a29a313f8/2e1ccfa8-8bce-4bb4-9d3d-716156df4d18"
-					(reference "#PWR0115")
+					(reference "#PWR0118")
 					(unit 1)
 				)
@@
 		(on_board yes)
 		(dnp no)
-		(property "Reference" "#PWR0128"
+		(property "Reference" "#PWR0131"
 			(at 267.97 142.24 0)
 			(effects
@@
 			(project "Main Board"
 				(path "/20aae4b7-3fb8-4924-82e8-1e7a29a313f8/2e1ccfa8-8bce-4bb4-9d3d-716156df4d18"
-					(reference "#PWR0128")
+					(reference "#PWR0131")
 					(unit 1)
 				)
@@
 		(on_board yes)
 		(dnp no)
-		(property "Reference" "#PWR0116"
+		(property "Reference" "#PWR0119"
 			(at 33.02 54.61 0)
 			(effects
@@
 			(project "Main Board"
 				(path "/20aae4b7-3fb8-4924-82e8-1e7a29a313f8/2e1ccfa8-8bce-4bb4-9d3d-716156df4d18"
-					(reference "#PWR0116")
+					(reference "#PWR0119")
 					(unit 1)
 				)
@@
 		(on_board yes)
 		(dnp no)
-		(property "Reference" "R83"
+		(property "Reference" "R87"
 			(at 146.05 54.61 90)
 			(effects
@@
 			(project "Main Board"
 				(path "/20aae4b7-3fb8-4924-82e8-1e7a29a313f8/2e1ccfa8-8bce-4bb4-9d3d-716156df4d18"
-					(reference "R83")
+					(reference "R87")
 					(unit 1)
 				)
@@
 		(on_board yes)
 		(dnp no)
-		(property "Reference" "R82"
+		(property "Reference" "R86"
 			(at 146.05 35.56 90)
 			(effects
@@
 			(project "Main Board"
 				(path "/20aae4b7-3fb8-4924-82e8-1e7a29a313f8/2e1ccfa8-8bce-4bb4-9d3d-716156df4d18"
-					(reference "R82")
+					(reference "R86")
 					(unit 1)
 				)
@@
 		(dnp no)
 		(fields_autoplaced yes)
-		(property "Reference" "#PWR0121"
+		(property "Reference" "#PWR0124"
 			(at 222.25 147.32 0)
 			(effects
@@
 			(project "Main Board"
 				(path "/20aae4b7-3fb8-4924-82e8-1e7a29a313f8/2e1ccfa8-8bce-4bb4-9d3d-716156df4d18"
-					(reference "#PWR0121")
+					(reference "#PWR0124")
 					(unit 1)
 				)
@@
 		(dnp no)
 		(fields_autoplaced yes)
-		(property "Reference" "R78"
+		(property "Reference" "R82"
 			(at 69.85 44.45 90)
 			(effects
@@
 			(project "Main Board"
 				(path "/20aae4b7-3fb8-4924-82e8-1e7a29a313f8/2e1ccfa8-8bce-4bb4-9d3d-716156df4d18"
-					(reference "R78")
+					(reference "R82")
 					(unit 1)
 				)
@@
 		(dnp no)
 		(fields_autoplaced yes)
-		(property "Reference" "#PWR0122"
+		(property "Reference" "#PWR0125"
 			(at 234.95 91.44 0)
 			(effects
@@
 			(project "Main Board"
 				(path "/20aae4b7-3fb8-4924-82e8-1e7a29a313f8/2e1ccfa8-8bce-4bb4-9d3d-716156df4d18"
-					(reference "#PWR0122")
+					(reference "#PWR0125")
 					(unit 1)
 				)
@@
 		(dnp no)
 		(fields_autoplaced yes)
-		(property "Reference" "#PWR0125"
+		(property "Reference" "#PWR0128"
 			(at 247.65 137.16 0)
 			(effects
@@
 			(project "Main Board"
 				(path "/20aae4b7-3fb8-4924-82e8-1e7a29a313f8/2e1ccfa8-8bce-4bb4-9d3d-716156df4d18"
-					(reference "#PWR0125")
+					(reference "#PWR0128")
 					(unit 1)
 				)
@@
 		(on_board yes)
 		(dnp no)
-		(property "Reference" "#PWR0127"
+		(property "Reference" "#PWR0130"
 			(at 265.43 152.4 0)
 			(effects
@@
 			(project "Main Board"
 				(path "/20aae4b7-3fb8-4924-82e8-1e7a29a313f8/2e1ccfa8-8bce-4bb4-9d3d-716156df4d18"
-					(reference "#PWR0127")
+					(reference "#PWR0130")
 					(unit 1)
 				)
@@
 		(dnp no)
 		(fields_autoplaced yes)
-		(property "Reference" "R86"
+		(property "Reference" "R90"
 			(at 237.49 68.5799 0)
 			(effects
@@
 			(project "Main Board"
 				(path "/20aae4b7-3fb8-4924-82e8-1e7a29a313f8/2e1ccfa8-8bce-4bb4-9d3d-716156df4d18"
-					(reference "R86")
+					(reference "R90")
 					(unit 1)
 				)
@@
 		(dnp no)
 		(fields_autoplaced yes)
-		(property "Reference" "#PWR0124"
+		(property "Reference" "#PWR0127"
 			(at 254 133.35 0)
 			(effects
@@
 			(project "Main Board"
 				(path "/20aae4b7-3fb8-4924-82e8-1e7a29a313f8/2e1ccfa8-8bce-4bb4-9d3d-716156df4d18"
-					(reference "#PWR0124")
+					(reference "#PWR0127")
 					(unit 1)
 				)
@@
 		(dnp no)
 		(fields_autoplaced yes)
-		(property "Reference" "#PWR0123"
+		(property "Reference" "#PWR0126"
 			(at 247.65 129.54 0)
 			(effects
@@
 			(project "Main Board"
 				(path "/20aae4b7-3fb8-4924-82e8-1e7a29a313f8/2e1ccfa8-8bce-4bb4-9d3d-716156df4d18"
-					(reference "#PWR0123")
+					(reference "#PWR0126")
 					(unit 1)
 				)
@@
 		(dnp no)
 		(fields_autoplaced yes)
-		(property "Reference" "#PWR0119"
+		(property "Reference" "#PWR0122"
 			(at 203.2 59.69 0)
 			(effects
@@
 			(project "Main Board"
 				(path "/20aae4b7-3fb8-4924-82e8-1e7a29a313f8/2e1ccfa8-8bce-4bb4-9d3d-716156df4d18"
-					(reference "#PWR0119")
+					(reference "#PWR0122")
 					(unit 1)
 				)
@@
 		(dnp no)
 		(fields_autoplaced yes)
-		(property "Reference" "R84"
+		(property "Reference" "R88"
 			(at 196.85 44.45 90)
 			(effects
@@
 			(project "Main Board"
 				(path "/20aae4b7-3fb8-4924-82e8-1e7a29a313f8/2e1ccfa8-8bce-4bb4-9d3d-716156df4d18"
-					(reference "R84")
+					(reference "R88")
 					(unit 1)
 				)
@@
 		(dnp no)
 		(fields_autoplaced yes)
-		(property "Reference" "#PWR0120"
+		(property "Reference" "#PWR0123"
 			(at 222.25 129.54 0)
 			(effects
@@
 			(project "Main Board"
 				(path "/20aae4b7-3fb8-4924-82e8-1e7a29a313f8/2e1ccfa8-8bce-4bb4-9d3d-716156df4d18"
-					(reference "#PWR0120")
+					(reference "#PWR0123")
 					(unit 1)
 				)
@@
 		(on_board yes)
 		(dnp no)
-		(property "Reference" "R80"
+		(property "Reference" "R84"
 			(at 133.35 54.61 90)
 			(effects
@@
 			(project "Main Board"
 				(path "/20aae4b7-3fb8-4924-82e8-1e7a29a313f8/2e1ccfa8-8bce-4bb4-9d3d-716156df4d18"
-					(reference "R80")
+					(reference "R84")
 					(unit 1)
 				)
@@
 		(on_board yes)
 		(dnp no)
-		(property "Reference" "R79"
+		(property "Reference" "R83"
 			(at 133.35 35.56 90)
 			(effects
@@
 			(project "Main Board"
 				(path "/20aae4b7-3fb8-4924-82e8-1e7a29a313f8/2e1ccfa8-8bce-4bb4-9d3d-716156df4d18"
-					(reference "R79")
+					(reference "R83")
 					(unit 1)
 				)

Commit message: New Resistor Selection Circuit
Parts:
- renumbered R80 to R85, R81 to R86, R82 to R87, R83 to R88, R84 to R89, R85 to R90, R86 to R91, R87 to R92, R88 to R93, R89 to R94, R90 to R95
Changed lines of the file:
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@@
 		(on_board yes)
 		(dnp no)
-		(property "Reference" "R85"
+		(property "Reference" "R90"
 			(at 139.7 73.66 90)
 			(effects
@@
 			(project "Main Board"
 				(path "/20aae4b7-3fb8-4924-82e8-1e7a29a313f8/2e1ccfa8-8bce-4bb4-9d3d-716156df4d18"
-					(reference "R85")
+					(reference "R90")
 					(unit 1)
 				)
@@
 		(dnp no)
 		(fields_autoplaced yes)
-		(property "Reference" "R89"
+		(property "Reference" "R94"
 			(at 237.49 57.1499 0)
 			(effects
@@
 			(project "Main Board"
 				(path "/20aae4b7-3fb8-4924-82e8-1e7a29a313f8/2e1ccfa8-8bce-4bb4-9d3d-716156df4d18"
-					(reference "R89")
+					(reference "R94")
 					(unit 1)
 				)
@@
 		(dnp no)
 		(fields_autoplaced yes)
-		(property "Reference" "#PWR0121"
+		(property "Reference" "#PWR0120"
 			(at 119.38 85.09 0)
 			(effects
@@
 			(project "Main Board"
 				(path "/20aae4b7-3fb8-4924-82e8-1e7a29a313f8/2e1ccfa8-8bce-4bb4-9d3d-716156df4d18"
-					(reference "#PWR0121")
+					(reference "#PWR0120")
 					(unit 1)
 				)
@@
 		(on_board yes)
 		(dnp no)
-		(property "Reference" "#PWR0120"
+		(property "Reference" "#PWR0119"
 			(at 38.1 54.61 0)
 			(effects
@@
 			(project "Main Board"
 				(path "/20aae4b7-3fb8-4924-82e8-1e7a29a313f8/2e1ccfa8-8bce-4bb4-9d3d-716156df4d18"
-					(reference "#PWR0120")
+					(reference "#PWR0119")
 					(unit 1)
 				)
@@
 		(dnp no)
 		(fields_autoplaced yes)
-		(property "Reference" "#PWR0129"
+		(property "Reference" "#PWR0128"
 			(at 265.43 124.46 0)
 			(effects
@@
 			(project "Main Board"
 				(path "/20aae4b7-3fb8-4924-82e8-1e7a29a313f8/2e1ccfa8-8bce-4bb4-9d3d-716156df4d18"
-					(reference "#PWR0129")
+					(reference "#PWR0128")
 					(unit 1)
 				)
@@
 		(on_board yes)
 		(dnp no)
-		(property "Reference" "R81"
+		(property "Reference" "R86"
 			(at 63.5 63.5 90)
 			(effects
@@
 			(project "Main Board"
 				(path "/20aae4b7-3fb8-4924-82e8-1e7a29a313f8/2e1ccfa8-8bce-4bb4-9d3d-716156df4d18"
-					(reference "R81")
+					(reference "R86")
 					(unit 1)
 				)
@@
 		(dnp no)
 		(fields_autoplaced yes)
-		(property "Reference" "R80"
+		(property "Reference" "R85"
 			(at 57.15 44.45 90)
 			(effects
@@
 			(project "Main Board"
 				(path "/20aae4b7-3fb8-4924-82e8-1e7a29a313f8/2e1ccfa8-8bce-4bb4-9d3d-716156df4d18"
-					(reference "R80")
+					(reference "R85")
 					(unit 1)
 				)
@@
 		(dnp no)
 		(fields_autoplaced yes)
-		(property "Reference" "#PWR0118"
+		(property "Reference" "#PWR0117"
 			(at 33.02 46.99 0)
 			(effects
@@
 			(project "Main Board"
 				(path "/20aae4b7-3fb8-4924-82e8-1e7a29a313f8/2e1ccfa8-8bce-4bb4-9d3d-716156df4d18"
-					(reference "#PWR0118")
+					(reference "#PWR0117")
 					(unit 1)
 				)
@@
 		(on_board yes)
 		(dnp no)
-		(property "Reference" "#PWR0131"
+		(property "Reference" "#PWR0130"
 			(at 267.97 142.24 0)
 			(effects
@@
 			(project "Main Board"
 				(path "/20aae4b7-3fb8-4924-82e8-1e7a29a313f8/2e1ccfa8-8bce-4bb4-9d3d-716156df4d18"
-					(reference "#PWR0131")
+					(reference "#PWR0130")
 					(unit 1)
 				)
@@
 		(on_board yes)
 		(dnp no)
-		(property "Reference" "#PWR0119"
+		(property "Reference" "#PWR0118"
 			(at 33.02 54.61 0)
 			(effects
@@
 			(project "Main Board"
 				(path "/20aae4b7-3fb8-4924-82e8-1e7a29a313f8/2e1ccfa8-8bce-4bb4-9d3d-716156df4d18"
-					(reference "#PWR0119")
+					(reference "#PWR0118")
 					(unit 1)
 				)
@@
 		(on_board yes)
 		(dnp no)
-		(property "Reference" "R87"
+		(property "Reference" "R92"
 			(at 146.05 54.61 90)
 			(effects
@@
 			(project "Main Board"
 				(path "/20aae4b7-3fb8-4924-82e8-1e7a29a313f8/2e1ccfa8-8bce-4bb4-9d3d-716156df4d18"
-					(reference "R87")
+					(reference "R92")
 					(unit 1)
 				)
@@
 		(on_board yes)
 		(dnp no)
-		(property "Reference" "R86"
+		(property "Reference" "R91"
 			(at 146.05 35.56 90)
 			(effects
@@
 			(project "Main Board"
 				(path "/20aae4b7-3fb8-4924-82e8-1e7a29a313f8/2e1ccfa8-8bce-4bb4-9d3d-716156df4d18"
-					(reference "R86")
+					(reference "R91")
 					(unit 1)
 				)
@@
 		(dnp no)
 		(fields_autoplaced yes)
-		(property "Reference" "#PWR0124"
+		(property "Reference" "#PWR0123"
 			(at 222.25 147.32 0)
 			(effects
@@
 			(project "Main Board"
 				(path "/20aae4b7-3fb8-4924-82e8-1e7a29a313f8/2e1ccfa8-8bce-4bb4-9d3d-716156df4d18"
-					(reference "#PWR0124")
+					(reference "#PWR0123")
 					(unit 1)
 				)
@@
 		(dnp no)
 		(fields_autoplaced yes)
-		(property "Reference" "R82"
+		(property "Reference" "R87"
 			(at 69.85 44.45 90)
 			(effects
@@
 			(project "Main Board"
 				(path "/20aae4b7-3fb8-4924-82e8-1e7a29a313f8/2e1ccfa8-8bce-4bb4-9d3d-716156df4d18"
-					(reference "R82")
+					(reference "R87")
 					(unit 1)
 				)
@@
 		(dnp no)
 		(fields_autoplaced yes)
-		(property "Reference" "#PWR0125"
+		(property "Reference" "#PWR0124"
 			(at 234.95 91.44 0)
 			(effects
@@
 			(project "Main Board"
 				(path "/20aae4b7-3fb8-4924-82e8-1e7a29a313f8/2e1ccfa8-8bce-4bb4-9d3d-716156df4d18"
-					(reference "#PWR0125")
+					(reference "#PWR0124")
 					(unit 1)
 				)
@@
 		(dnp no)
 		(fields_autoplaced yes)
-		(property "Reference" "#PWR0128"
+		(property "Reference" "#PWR0127"
 			(at 247.65 137.16 0)
 			(effects
@@
 			(project "Main Board"
 				(path "/20aae4b7-3fb8-4924-82e8-1e7a29a313f8/2e1ccfa8-8bce-4bb4-9d3d-716156df4d18"
-					(reference "#PWR0128")
+					(reference "#PWR0127")
 					(unit 1)
 				)
@@
 		(on_board yes)
 		(dnp no)
-		(property "Reference" "#PWR0130"
+		(property "Reference" "#PWR0129"
 			(at 265.43 152.4 0)
 			(effects
@@
 			(project "Main Board"
 				(path "/20aae4b7-3fb8-4924-82e8-1e7a29a313f8/2e1ccfa8-8bce-4bb4-9d3d-716156df4d18"
-					(reference "#PWR0130")
+					(reference "#PWR0129")
 					(unit 1)
 				)
@@
 		(dnp no)
 		(fields_autoplaced yes)
-		(property "Reference" "R90"
+		(property "Reference" "R95"
 			(at 237.49 68.5799 0)
 			(effects
@@
 			(project "Main Board"
 				(path "/20aae4b7-3fb8-4924-82e8-1e7a29a313f8/2e1ccfa8-8bce-4bb4-9d3d-716156df4d18"
-					(reference "R90")
+					(reference "R95")
 					(unit 1)
 				)
@@
 		(dnp no)
 		(fields_autoplaced yes)
-		(property "Reference" "#PWR0127"
+		(property "Reference" "#PWR0126"
 			(at 254 133.35 0)
 			(effects
@@
 			(project "Main Board"
 				(path "/20aae4b7-3fb8-4924-82e8-1e7a29a313f8/2e1ccfa8-8bce-4bb4-9d3d-716156df4d18"
-					(reference "#PWR0127")
+					(reference "#PWR0126")
 					(unit 1)
 				)
@@
 		(dnp no)
 		(fields_autoplaced yes)
-		(property "Reference" "#PWR0126"
+		(property "Reference" "#PWR0125"
 			(at 247.65 129.54 0)
 			(effects
@@
 			(project "Main Board"
 				(path "/20aae4b7-3fb8-4924-82e8-1e7a29a313f8/2e1ccfa8-8bce-4bb4-9d3d-716156df4d18"
-					(reference "#PWR0126")
+					(reference "#PWR0125")
 					(unit 1)
 				)
@@
 		(dnp no)
 		(fields_autoplaced yes)
-		(property "Reference" "#PWR0122"
+		(property "Reference" "#PWR0121"
 			(at 203.2 59.69 0)
 			(effects
@@
 			(project "Main Board"
 				(path "/20aae4b7-3fb8-4924-82e8-1e7a29a313f8/2e1ccfa8-8bce-4bb4-9d3d-716156df4d18"
-					(reference "#PWR0122")
+					(reference "#PWR0121")
 					(unit 1)
 				)
@@
 		(dnp no)
 		(fields_autoplaced yes)
-		(property "Reference" "R88"
+		(property "Reference" "R93"
 			(at 196.85 44.45 90)
 			(effects
@@
 			(project "Main Board"
 				(path "/20aae4b7-3fb8-4924-82e8-1e7a29a313f8/2e1ccfa8-8bce-4bb4-9d3d-716156df4d18"
-					(reference "R88")
+					(reference "R93")
 					(unit 1)
 				)
@@
 		(dnp no)
 		(fields_autoplaced yes)
-		(property "Reference" "#PWR0123"
+		(property "Reference" "#PWR0122"
 			(at 222.25 129.54 0)
 			(effects
@@
 			(project "Main Board"
 				(path "/20aae4b7-3fb8-4924-82e8-1e7a29a313f8/2e1ccfa8-8bce-4bb4-9d3d-716156df4d18"
-					(reference "#PWR0123")
+					(reference "#PWR0122")
 					(unit 1)
 				)
@@
 		(on_board yes)
 		(dnp no)
-		(property "Reference" "R84"
+		(property "Reference" "R89"
 			(at 133.35 54.61 90)
 			(effects
@@
 			(project "Main Board"
 				(path "/20aae4b7-3fb8-4924-82e8-1e7a29a313f8/2e1ccfa8-8bce-4bb4-9d3d-716156df4d18"
-					(reference "R84")
+					(reference "R89")
 					(unit 1)
 				)
@@
 		(on_board yes)
 		(dnp no)
-		(property "Reference" "R83"
+		(property "Reference" "R88"
 			(at 133.35 35.56 90)
 			(effects
@@
 			(project "Main Board"
 				(path "/20aae4b7-3fb8-4924-82e8-1e7a29a313f8/2e1ccfa8-8bce-4bb4-9d3d-716156df4d18"
-					(reference "R83")
-					(unit 1)
-				)
+					(reference "R88")
+					(unit 1)
+				)
