File: Circuit/Bridge.kicad_sch (KiCad schematic)
At the start: 42 parts, among them K2 AGQ200A12, Q4 TIP41C, Q5 TIP42C, Q6 TIP41C, Q7 TIP42C, U10 OPA2376xxD, U6 OPA2197xD, U7 ULN2003, U8 OPA2197xD, U9 DG201

Commit message: Adjustments
Connections:
- net GUARD: no longer R40.1, U8.2 (-)
- new net: R40.1, U8.2 (-)
Other:
- moved on the sheet: C19, C20, C23, JP2, R40, U10C, U6C, U8A
