File: Circuit/Source.kicad_sch (KiCad schematic)
At the start: 41 parts, among them K1 AGQ200A12, Q1 2N7002, Q2 TIP41C, Q3 TIP42C, U2 DG201, U3 OPA2197xD, U4 OPA2197xD, U5 OPA2197xD

Commit message: Adjustments
Parts:
- removed JP1: SolderJumper_2_Open, Jumper:SolderJumper-2_P1.3mm_Open_RoundedPad1.0x1.5mm, symbol Jumper:SolderJumper_2_Open
- added D15: BAV99, Package_TO_SOT_SMD:SOT-23, symbol Diode:BAV99
Connections:
- net +18V: now also D15.2 (A)
- net -18V: now also D15.1 (K)
- net at Q2.3 (E), Q3.3 (E), R22.2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: now also D15.3 (K)
- net at R29.2, R30.2: now also K1.4; no longer K1.2
- net at R31.2, R32.2: now also K1.2; no longer K1.4
Other:
- note added: "Bias range: ±10VDC Gain: ~6.5"
- note removed: "Bias range: ±10V Gain: ~6.5"
- moved on the sheet: R25, R26, R27, R28, R29, R30, R31, R32
