File: Circuit/Power.kicad_sch (KiCad schematic)
At the start: 12 parts, among them J9 Conn_01x05_Pin

Commit message: Adjustments
Other:
- moved on the sheet: C50, C51, C52, C53, D10, D11, D12, D13, D14, FB1, J9, R96

Commit message: Final Touches
Connections:
- net +12V: now also J9.4 (Pin_4); no longer J9.2 (Pin_2)
- net +18V: now also J9.5 (Pin_5); no longer J9.1 (Pin_1)
- net -18V: now also J9.1 (Pin_1); no longer J9.5 (Pin_5)
- net GND: now also J9.2 (Pin_2); no longer J9.4 (Pin_4)
Changed lines of the file:
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@@
 		(lib_id "Connector:Conn_01x05_Pin")
 		(at 50.8 88.9 0)
+		(mirror x)
 		(unit 1)
 		(body_style 1)
@@
 		(in_pos_files yes)
 		(dnp no)
-		(fields_autoplaced yes)
 		(property "Reference" "J9"
-			(at 51.435 78.74 0)
+			(at 50.8 77.47 0)
 			(show_name no)
 			(do_not_autoplace no)
@@
 		)
 		(property "Value" "Conn_01x05_Pin"
-			(at 51.435 81.28 0)
+			(at 50.8 80.01 0)
 			(show_name no)
 			(do_not_autoplace no)
